Commit message: removed dep on iiwaconfig + updated urdf

File: config/robot_properties_kuka/iiwa.urdf (robot description, URDF)
Before this commit: robot KUKAiiwa, 9 links, 8 joints
Links:
- added link world
- link L1: mass 4.00000 -> 3.94781; geometry collision mesh filename=package://meshes/stl/iiwa_link_1.stl; visual mesh filename=package://meshes/stl/iiwa_link_1.stl
- link L2: mass 4.00000 -> 4; geometry collision mesh filename=package://meshes/stl/iiwa_link_2.stl; visual mesh filename=package://meshes/stl/iiwa_link_2.stl
- link L3: mass 4.00000 -> 3; geometry collision mesh filename=package://meshes/stl/iiwa_link_3.stl; visual mesh filename=package://meshes/stl/iiwa_link_3.stl
- link L4: mass 4.00000 -> 2.7; geometry collision mesh filename=package://meshes/stl/iiwa_link_4.stl; visual mesh filename=package://meshes/stl/iiwa_link_4.stl
- link L5: mass 3.00000 -> 1.7; geometry collision mesh filename=package://meshes/stl/iiwa_link_5.stl; visual mesh filename=package://meshes/stl/iiwa_link_5.stl
- link L6: mass 2.00000 -> 1.8; geometry collision mesh filename=package://meshes/stl/iiwa_link_6.stl; visual mesh filename=package://meshes/stl/iiwa_link_6.stl
- link L7: mass 1.00000 -> 0.3; geometry collision mesh filename=package://meshes/stl/iiwa_link_7.stl; visual mesh filename=package://meshes/stl/iiwa_link_7.stl
- link contact: geometry collision mesh filename=package://meshes/tennis_ball_smaller.obj; visual mesh filename=package://meshes/tennis_ball_smaller.obj
- link iiwa_base: mass 8.00000 -> 5; geometry collision mesh filename=package://meshes/stl/iiwa_base.stl; visual mesh filename=package://meshes/stl/iiwa_base.stl
Joints:
- added joint A0: type fixed, parent world, child iiwa_base, origin xyz=0 0 0 rpy=0 0 0
- joint A1: limit effort=30 velocity=1.0 -> lower=-2.96706 upper=2.96706 effort=320 velocity=1.48353
